Commit message: Fully connected Gazebo and RViz; completed the whole process of dual_ur5_motion.py, especially the gripper part.

File: ur_description/urdf/ur5_robot.urdf (robot description, URDF)
Before this commit: robot ur5, 32 links, 31 joints
Joints:
- joint left_rh_l1: mimic joint=left_rh_p12_rn multiplier=1.0 -> (none)
- joint left_rh_l2: mimic joint=left_rh_p12_rn multiplier=0.9090909 -> (none)
- joint left_rh_r2: mimic joint=left_rh_p12_rn multiplier=0.9090909 -> (none)
- joint right_rh_l1: mimic joint=right_rh_p12_rn multiplier=1.0 -> (none)
- joint right_rh_l2: mimic joint=right_rh_p12_rn multiplier=0.9090909 -> (none)
- joint right_rh_r2: mimic joint=right_rh_p12_rn multiplier=0.9090909 -> (none)
