Commit message: Tested three different time parameterization algorithms, but found out that computeCartesianPath doesn't support TP algorithms other than the hard-coded IPTP; Removed obsolete packages.

File: ur_description/urdf/ur5_robot_backup_original_range.urdf (robot description, URDF)
Before this commit: robot ur5, 32 links, 31 joints
Joints:
- joint left_elbow_joint: limit lower=-7.854 upper=4.712 effort=150.0 velocity=3.15 -> lower=-3.14159265359 upper=3.14159265359 effort=150.0 velocity=3.15
- joint left_shoulder_lift_joint: limit lower=-5.498 upper=7.069 effort=150.0 velocity=3.15 -> lower=-6.28318530718 upper=6.28318530718 effort=150.0 velocity=3.15
- joint left_wrist_2_joint: limit lower=-7.854 upper=4.712 effort=28.0 velocity=3.2 -> lower=-6.28318530718 upper=6.28318530718 effort=28.0 velocity=3.2
- joint right_elbow_joint: limit lower=-4.712 upper=7.854 effort=150.0 velocity=3.15 -> lower=-3.14159265359 upper=3.14159265359 effort=150.0 velocity=3.15
- joint right_shoulder_lift_joint: limit lower=-3.927 upper=8.639 effort=150.0 velocity=3.15 -> lower=-6.28318530718 upper=6.28318530718 effort=150.0 velocity=3.15
- joint right_wrist_1_joint: limit lower=-3.1415926 upper=9.425 effort=28.0 velocity=3.2 -> lower=-6.28318530718 upper=6.28318530718 effort=28.0 velocity=3.2
- joint right_wrist_2_joint: limit lower=-4.712 upper=7.854 effort=28.0 velocity=3.2 -> lower=-6.28318530718 upper=6.28318530718 effort=28.0 velocity=3.2
