Commit message: Incorporate inspire-robot's left and right hands' URDF models. Enable Gazebo control and visualization.

File: ur_description/urdf/ur5_robot_with_hands.urdf (robot description, URDF)
Before this commit: robot ur5, 36 links, 35 joints
Links:
- removed link base
- added link left_hand_base
- added link link1, mass 0.00330630285835291; collision mesh filename=package://inspire_hand_description/meshes/left/link1.STL; visual mesh filename=package://inspire_hand_description/meshes/left/link1.STL
- added link link11, mass 0.00453366979354947; collision mesh filename=package://inspire_hand_description/meshes/left/link11.STL; visual mesh filename=package://inspire_hand_description/meshes/left/link11.STL
- added link link111, mass 0.226288892912552; collision mesh filename=package://inspire_hand_description/meshes/left/link111.STL; visual mesh filename=package://inspire_hand_description/meshes/left/link111.STL
- added link link2, mass 0.00330621735666597; collision mesh filename=package://inspire_hand_description/meshes/left/link2.STL; visual mesh filename=package://inspire_hand_description/meshes/left/link2.STL
- added link link22, mass 0.00453367027223764; collision mesh filename=package://inspire_hand_description/meshes/left/link22.STL; visual mesh filename=package://inspire_hand_description/meshes/left/link22.STL
- added link link3, mass 0.00330616517571661; collision mesh filename=package://inspire_hand_description/meshes/left/link3.STL; visual mesh filename=package://inspire_hand_description/meshes/left/link3.STL
- added link link33, mass 0.00453366946672897; collision mesh filename=package://inspire_hand_description/meshes/left/link33.STL; visual mesh filename=package://inspire_hand_description/meshes/left/link33.STL
- added link link4, mass 0.00330630460851054; collision mesh filename=package://inspire_hand_description/meshes/left/link4.STL; visual mesh filename=package://inspire_hand_description/meshes/left/link4.STL
- added link link44, mass 0.00356888715893842; collision mesh filename=package://inspire_hand_description/meshes/left/link44.STL; visual mesh filename=package://inspire_hand_description/meshes/left/link44.STL
- added link link5, mass 0.00487393910083768; collision mesh filename=package://inspire_hand_description/meshes/left/link5.STL; visual mesh filename=package://inspire_hand_description/meshes/left/link5.STL
- added link link51, mass 0.00652741708580189; collision mesh filename=package://inspire_hand_description/meshes/left/link51.STL; visual mesh filename=package://inspire_hand_description/meshes/left/link51.STL
- added link link52, mass 0.00226947954597765; collision mesh filename=package://inspire_hand_description/meshes/left/link52.STL; visual mesh filename=package://inspire_hand_description/meshes/left/link52.STL
- added link link53, mass 0.00330869122519449; collision mesh filename=package://inspire_hand_description/meshes/left/link53.STL; visual mesh filename=package://inspire_hand_description/meshes/left/link53.STL
- added link right_hand_base
- link Link1: geometry collision mesh filename=package://inspire_hand_description/meshes/right/Link1.STL; visual mesh filename=package://inspire_hand_description/meshes/right/Link1.STL
- link Link11: geometry collision mesh filename=package://inspire_hand_description/meshes/right/Link11.STL; visual mesh filename=package://inspire_hand_description/meshes/right/Link11.STL
- link Link111: geometry collision mesh filename=package://inspire_hand_description/meshes/right/Link111.STL; visual mesh filename=package://inspire_hand_description/meshes/right/Link111.STL
- link Link2: geometry collision mesh filename=package://inspire_hand_description/meshes/right/Link2.STL; visual mesh filename=package://inspire_hand_description/meshes/right/Link2.STL
- link Link22: geometry collision mesh filename=package://inspire_hand_description/meshes/right/Link22.STL; visual mesh filename=package://inspire_hand_description/meshes/right/Link22.STL
- link Link3: geometry collision mesh filename=package://inspire_hand_description/meshes/right/Link3.STL; visual mesh filename=package://inspire_hand_description/meshes/right/Link3.STL
- link Link33: geometry collision mesh filename=package://inspire_hand_description/meshes/right/Link33.STL; visual mesh filename=package://inspire_hand_description/meshes/right/Link33.STL
- link Link4: geometry collision mesh filename=package://inspire_hand_description/meshes/right/Link4.STL; visual mesh filename=package://inspire_hand_description/meshes/right/Link4.STL
- link Link44: geometry collision mesh filename=package://inspire_hand_description/meshes/right/Link44.STL; visual mesh filename=package://inspire_hand_description/meshes/right/Link44.STL
- link Link5: geometry collision mesh filename=package://inspire_hand_description/meshes/right/Link5.STL; visual mesh filename=package://inspire_hand_description/meshes/right/Link5.STL
- link Link51: geometry collision mesh filename=package://inspire_hand_description/meshes/right/Link51.STL; visual mesh filename=package://inspire_hand_description/meshes/right/Link51.STL
- link Link52: geometry collision mesh filename=package://inspire_hand_description/meshes/right/Link52.STL; visual mesh filename=package://inspire_hand_description/meshes/right/Link52.STL
- link Link53: geometry collision mesh filename=package://inspire_hand_description/meshes/right/Link53.STL; visual mesh filename=package://inspire_hand_description/meshes/right/Link53.STL
Joints:
- added joint left_gripper_joint: type fixed, parent left_ee_link, child left_hand_base, origin xyz=0 0 0 rpy=3.1415 -1.5707 0
- added joint link1: type revolute, parent link111, child link1, origin xyz=0.0068852 -0.0077547 -0.08206 rpy=-1.4604 1.2485 -1.466, axis 0 0 1, limit lower=-1 upper=0 effort=1 velocity=1
- added joint link11: type revolute, parent link1, child link11, origin xyz=0.032132 0 0 rpy=-5.2101E-10 -2.8366E-11 -0.05439, axis 0 0 1, limit lower=-2 upper=0 effort=1 velocity=1
- added joint link111_shift: type fixed, parent left_hand_base, child link111, origin xyz=-0.00850 -0.0190 0.0404 rpy=3.1415 0 -1.5707
- added joint link2: type revolute, parent link111, child link2, origin xyz=-0.012436 -0.0077547 -0.082423 rpy=-1.5708 1.4093 -1.5708, axis 0 0 1, limit lower=-1 upper=0 effort=1 velocity=1
- added joint link22: type revolute, parent link2, child link22, origin xyz=0.032132 0 0 rpy=-5.0853E-10 -1.1686E-10 -0.22588, axis 0 0 1, limit lower=-2 upper=0 effort=1 velocity=1
- added joint link3: type revolute, parent link111, child link3, origin xyz=-0.031665 -0.0077547 -0.08192 rpy=-1.9857 1.4406 -1.9826, axis 0 0 1, limit lower=-1 upper=0 effort=1 velocity=1
- added joint link33: type revolute, parent link3, child link33, origin xyz=0.032132 0 0 rpy=-5.0314E-10 -1.3824E-10 -0.26815, axis 0 0 1, limit lower=-2 upper=0 effort=1 velocity=1
- added joint link4: type revolute, parent link111, child link4, origin xyz=-0.050841 -0.0077547 -0.08041 rpy=-2.0186 1.327 -2.007, axis 0 0 1, limit lower=-1 upper=0 effort=1 velocity=1
- added joint link44: type revolute, parent link4, child link44, origin xyz=0.032132 0 0 rpy=-5.1334E-10 -9.3483E-11 -0.18013, axis 0 0 1, limit lower=-2 upper=0 effort=1 velocity=1
- added joint link5: type revolute, parent link111, child link5, origin xyz=0.0010638 -0.025 -0.0059231 rpy=-1.5708 -2.455E-15 2.3555, axis 0 1 0, limit lower=0 upper=1 effort=1 velocity=1
- added joint link51: type revolute, parent link5, child link51, origin xyz=-0.0115 -0.00075 0 rpy=-1.4988E-15 -5.5511E-17 1.8988, axis 0 0 1, limit lower=0 upper=1 effort=1 velocity=1
- added joint link52: type revolute, parent link51, child link52, origin xyz=0.056001 0 0 rpy=-1.3323E-15 -2.7756E-17 -3.0416, axis 0 0 1, limit lower=-1 upper=0 effort=1 velocity=1
- added joint link53: type revolute, parent link52, child link53, origin xyz=-0.022653 0 0 rpy=1.2712E-14 -9.7145E-17 2.856, axis 0 0 1, limit lower=-1 upper=0 effort=1 velocity=1
- joint Link111_shift: parent base -> right_hand_base
- joint right_gripper_joint: child base -> right_hand_base

Commit message: Update the parts of Inspire hands in UR5(_with_hands) and YuMi(_with_hands) models.   - The joint limits of inspire hands in UR5 and YuMi's URDFs are not in consistent with the updated Inspire hands' URDFs as well as the optimization code, which causes joint-value-out-of-bounds error.

File: ur_description/urdf/ur5_robot_with_hands.urdf (robot description, URDF)
Before this commit: robot ur5, 50 links, 49 joints
Joints:
- joint link1: limit lower=-1 upper=0 effort=1 velocity=1 -> lower=-1.6 upper=0 effort=1 velocity=1
- joint link11: limit lower=-2 upper=0 effort=1 velocity=1 -> lower=-1.7 upper=0 effort=1 velocity=1
- joint link2: limit lower=-1 upper=0 effort=1 velocity=1 -> lower=-1.6 upper=0 effort=1 velocity=1
- joint link22: limit lower=-2 upper=0 effort=1 velocity=1 -> lower=-1.7 upper=0 effort=1 velocity=1
- joint link3: limit lower=-1 upper=0 effort=1 velocity=1 -> lower=-1.6 upper=0 effort=1 velocity=1
- joint link33: limit lower=-2 upper=0 effort=1 velocity=1 -> lower=-1.7 upper=0 effort=1 velocity=1
- joint link4: limit lower=-1 upper=0 effort=1 velocity=1 -> lower=-1.6 upper=0 effort=1 velocity=1
- joint link44: limit lower=-2 upper=0 effort=1 velocity=1 -> lower=-1.7 upper=0 effort=1 velocity=1
- joint link5: axis 0 1 0 -> 0 -1 0; limit lower=0 upper=1 effort=1 velocity=1 -> lower=-1.0 upper=0.3 effort=1 velocity=1
- joint link51: axis 0 0 1 -> 0 0 -1; limit lower=0 upper=1 effort=1 velocity=1 -> lower=0 upper=0.4 effort=1 velocity=1
- joint link52: limit lower=-1 upper=0 effort=1 velocity=1 -> lower=-0.4 upper=0 effort=1 velocity=1

File: yumi_description/urdf/yumi_with_hands.urdf (robot description, URDF)
Before this commit: robot yumi, 45 links, 44 joints
Joints:
- joint link1: limit lower=-1 upper=0 effort=1 velocity=1 -> lower=-1.6 upper=0 effort=1 velocity=1
- joint link11: limit lower=-2 upper=0 effort=1 velocity=1 -> lower=-1.7 upper=0 effort=1 velocity=1
- joint link2: limit lower=-1 upper=0 effort=1 velocity=1 -> lower=-1.6 upper=0 effort=1 velocity=1
- joint link22: limit lower=-2 upper=0 effort=1 velocity=1 -> lower=-1.7 upper=0 effort=1 velocity=1
- joint link3: limit lower=-1 upper=0 effort=1 velocity=1 -> lower=-1.6 upper=0 effort=1 velocity=1
- joint link33: limit lower=-2 upper=0 effort=1 velocity=1 -> lower=-1.7 upper=0 effort=1 velocity=1
- joint link4: limit lower=-1 upper=0 effort=1 velocity=1 -> lower=-1.6 upper=0 effort=1 velocity=1
- joint link44: limit lower=-2 upper=0 effort=1 velocity=1 -> lower=-1.7 upper=0 effort=1 velocity=1
- joint link5: axis 0 1 0 -> 0 -1 0; limit lower=0 upper=1 effort=1 velocity=1 -> lower=-1.0 upper=0.3 effort=1 velocity=1
- joint link51: axis 0 0 1 -> 0 0 -1; limit lower=0 upper=1 effort=1 velocity=1 -> lower=0 upper=0.4 effort=1 velocity=1
- joint link52: limit lower=-1 upper=0 effort=1 velocity=1 -> lower=-0.4 upper=0 effort=1 velocity=1
