Commit message: Add a better located base reference to the URDF hand model for convenience.

File: inspire_hand_description/robots/urdf-five3.urdf (robot description, URDF)
Before this commit: robot inspire_hand_description, 13 links, 12 joints
Links:
- added link base
Joints:
- added joint Link111_shift: type fixed, parent base, child Link111, origin xyz=-0.00850 0.0180 0.0404 rpy=1.5707 -1.5707 0
