Commit message: Modify the left Inspire hand's URDF to match the right hand's limits.

File: inspire_hand_description/robots/inspire_hand_left.urdf (robot description, URDF)
Before this commit: robot inspire_hand_left, 14 links, 13 joints
Joints:
- joint link1: limit lower=-1 upper=0 effort=1 velocity=1 -> lower=-1.6 upper=0 effort=1 velocity=1
- joint link11: limit lower=-2 upper=0 effort=1 velocity=1 -> lower=-1.7 upper=0 effort=1 velocity=1
- joint link2: limit lower=-1 upper=0 effort=1 velocity=1 -> lower=-1.6 upper=0 effort=1 velocity=1
- joint link22: limit lower=-2 upper=0 effort=1 velocity=1 -> lower=-1.7 upper=0 effort=1 velocity=1
- joint link3: limit lower=-1 upper=0 effort=1 velocity=1 -> lower=-1.6 upper=0 effort=1 velocity=1
- joint link33: limit lower=-2 upper=0 effort=1 velocity=1 -> lower=-1.7 upper=0 effort=1 velocity=1
- joint link4: limit lower=-1 upper=0 effort=1 velocity=1 -> lower=-1.6 upper=0 effort=1 velocity=1
- joint link44: limit lower=-2 upper=0 effort=1 velocity=1 -> lower=-1.7 upper=0 effort=1 velocity=1
- joint link5: axis 0 1 0 -> 0 -1 0; limit lower=0 upper=1 effort=1 velocity=1 -> lower=-1.0 upper=0.3 effort=1 velocity=1
- joint link51: axis 0 0 1 -> 0 0 -1; limit lower=0 upper=1 effort=1 velocity=1 -> lower=0 upper=0.4 effort=1 velocity=1
- joint link52: limit lower=-1 upper=0 effort=1 velocity=1 -> lower=-0.4 upper=0 effort=1 velocity=1
