Commit message: Set the reference link of human hand model configurable for visualization.

File: arm_hand_retargeting/urdf/human_hand_model.urdf (robot description, URDF)
Before this commit: robot human_hand_model, 2 links, 0 joints
Links:
- removed link right_palm
- removed link world
- added link tmp_index_finger_DP_link; visual box size=0.01 0.015 0.02
- added link tmp_index_finger_IP_link; visual box size=0.01 0.015 0.03
- added link tmp_index_finger_PP_link; visual box size=0.01 0.015 0.04
- added link tmp_index_finger_virtual_link
- added link tmp_little_finger_DP_link; visual box size=0.01 0.015 0.01
- added link tmp_little_finger_IP_link; visual box size=0.01 0.015 0.02
- added link tmp_little_finger_PP_link; visual box size=0.01 0.015 0.03
- added link tmp_little_finger_virtual_link
- added link tmp_middle_finger_DP_link; visual box size=0.01 0.015 0.021
- added link tmp_middle_finger_IP_link; visual box size=0.01 0.015 0.032
- added link tmp_middle_finger_PP_link; visual box size=0.01 0.015 0.043
- added link tmp_middle_finger_virtual_link
- added link tmp_palm; visual box size=0.01 0.1 0.15
- added link tmp_ring_finger_DP_link; visual box size=0.01 0.015 0.02
- added link tmp_ring_finger_IP_link; visual box size=0.01 0.015 0.03
- added link tmp_ring_finger_PP_link; visual box size=0.01 0.015 0.04
- added link tmp_ring_finger_virtual_link
- added link tmp_thumb_DP_link; visual box size=0.01 0.015 0.02
- added link tmp_thumb_IP_link; visual box size=0.01 0.015 0.03
- added link tmp_thumb_PP_link; visual box size=0.01 0.015 0.05
- added link tmp_thumb_virtual_link_1
- added link tmp_thumb_virtual_link_2
Joints:
- added joint tmp_index_finger_DIP_joint: type revolute, parent tmp_index_finger_IP_link, child tmp_index_finger_DP_link, origin xyz=0 0 0.03 rpy=0 0 0, axis 0 1 0, limit lower=0 upper=1.57079632679 effort=100 velocity=10.0
- added joint tmp_index_finger_MCP_abduction_joint: type revolute, parent tmp_palm, child tmp_index_finger_virtual_link, origin xyz=0.0 0.0425 0.15 rpy=0 0 0, axis 1 0 0, limit lower=-0.174532925199 upper=0.174532925199 effort=100 velocity=10.0
- added joint tmp_index_finger_MCP_flexion_joint: type revolute, parent tmp_index_finger_virtual_link, child tmp_index_finger_PP_link, origin xyz=0 0 0 rpy=0 0 0, axis 0 1 0, limit lower=0 upper=1.57079632679 effort=100 velocity=10.0
- added joint tmp_index_finger_PIP_joint: type revolute, parent tmp_index_finger_PP_link, child tmp_index_finger_IP_link, origin xyz=0 0 0.04 rpy=0 0 0, axis 0 1 0, limit lower=0 upper=1.57079632679 effort=100 velocity=10.0
- added joint tmp_little_finger_DIP_joint: type revolute, parent tmp_little_finger_IP_link, child tmp_little_finger_DP_link, origin xyz=0 0 0.02 rpy=0 0 0, axis 0 1 0, limit lower=0 upper=1.57079632679 effort=100 velocity=10.0
- added joint tmp_little_finger_MCP_abduction_joint: type revolute, parent tmp_palm, child tmp_little_finger_virtual_link, origin xyz=0.0 -0.0425 0.15 rpy=0 0 0, axis 1 0 0, limit lower=-0.174532925199 upper=0.174532925199 effort=100 velocity=10.0
- added joint tmp_little_finger_MCP_flexion_joint: type revolute, parent tmp_little_finger_virtual_link, child tmp_little_finger_PP_link, origin xyz=0 0 0 rpy=0 0 0, axis 0 1 0, limit lower=0 upper=1.57079632679 effort=100 velocity=10.0
- added joint tmp_little_finger_PIP_joint: type revolute, parent tmp_little_finger_PP_link, child tmp_little_finger_IP_link, origin xyz=0 0 0.03 rpy=0 0 0, axis 0 1 0, limit lower=0 upper=1.57079632679 effort=100 velocity=10.0
- added joint tmp_middle_finger_DIP_joint: type revolute, parent tmp_middle_finger_IP_link, child tmp_middle_finger_DP_link, origin xyz=0 0 0.032 rpy=0 0 0, axis 0 1 0, limit lower=0 upper=1.57079632679 effort=100 velocity=10.0
- added joint tmp_middle_finger_MCP_abduction_joint: type revolute, parent tmp_palm, child tmp_middle_finger_virtual_link, origin xyz=0.0 0.0175 0.15 rpy=0 0 0, axis 1 0 0, limit lower=-0.174532925199 upper=0.174532925199 effort=100 velocity=10.0
- added joint tmp_middle_finger_MCP_flexion_joint: type revolute, parent tmp_middle_finger_virtual_link, child tmp_middle_finger_PP_link, origin xyz=0 0 0 rpy=0 0 0, axis 0 1 0, limit lower=0 upper=1.57079632679 effort=100 velocity=10.0
- added joint tmp_middle_finger_PIP_joint: type revolute, parent tmp_middle_finger_PP_link, child tmp_middle_finger_IP_link, origin xyz=0 0 0.043 rpy=0 0 0, axis 0 1 0, limit lower=0 upper=1.57079632679 effort=100 velocity=10.0
- added joint tmp_palm_joint: type fixed, parent not_world, child tmp_palm, origin xyz=0 0 0 rpy=0 0 0
- added joint tmp_ring_finger_DIP_joint: type revolute, parent tmp_ring_finger_IP_link, child tmp_ring_finger_DP_link, origin xyz=0 0 0.03 rpy=0 0 0, axis 0 1 0, limit lower=0 upper=1.57079632679 effort=100 velocity=10.0
- added joint tmp_ring_finger_MCP_abduction_joint: type revolute, parent tmp_palm, child tmp_ring_finger_virtual_link, origin xyz=0.0 -0.0175 0.15 rpy=0 0 0, axis 1 0 0, limit lower=-0.174532925199 upper=0.174532925199 effort=100 velocity=10.0
- added joint tmp_ring_finger_MCP_flexion_joint: type revolute, parent tmp_ring_finger_virtual_link, child tmp_ring_finger_PP_link, origin xyz=0 0 0 rpy=0 0 0, axis 0 1 0, limit lower=0 upper=1.57079632679 effort=100 velocity=10.0
- added joint tmp_ring_finger_PIP_joint: type revolute, parent tmp_ring_finger_PP_link, child tmp_ring_finger_IP_link, origin xyz=0 0 0.04 rpy=0 0 0, axis 0 1 0, limit lower=0 upper=1.57079632679 effort=100 velocity=10.0
- added joint tmp_thumb_DIP_joint: type revolute, parent tmp_thumb_IP_link, child tmp_thumb_DP_link, origin xyz=0 0 0.03 rpy=0 0 0, axis 0 1 0, limit lower=0 upper=1.57079632679 effort=100 velocity=10.0
- added joint tmp_thumb_MCP_joint_1: type revolute, parent tmp_palm, child tmp_thumb_virtual_link_1, origin xyz=0.0 0.05 0.0 rpy=0 0 0, axis -1 0 0, limit lower=0.0 upper=0.349065850399 effort=100 velocity=10.0
- added joint tmp_thumb_MCP_joint_2: type revolute, parent tmp_thumb_virtual_link_1, child tmp_thumb_PP_link, origin xyz=0 0 0 rpy=0 0 0, axis 0 0 -1, limit lower=0 upper=1.74532925199 effort=100 velocity=10.0
- added joint tmp_thumb_PIP_joint_1: type revolute, parent tmp_thumb_PP_link, child tmp_thumb_virtual_link_2, origin xyz=0 0 0.05 rpy=0 0 0, axis 1 0 0, limit lower=0 upper=0.785398163397 effort=100 velocity=10.0
- added joint tmp_thumb_PIP_joint_2: type revolute, parent tmp_thumb_virtual_link_2, child tmp_thumb_IP_link, origin xyz=0 0 0 rpy=0 0 0, axis 0 1 0, limit lower=0 upper=1.57079632679 effort=100 velocity=10.0

File: arm_hand_retargeting/urdf/human_hand_model.urdf.xacro (robot description, xacro)
@@ -2,6 +2,8 @@
 <robot xmlns:xacro="http://wiki.ros.org/xacro"
              name="human_hand_model" >
+  <!-- Configurable arguments -->
+  <xacro:arg name="prefix" default="right" />
+  <xacro:arg name="parent" default="world" />
   <!-- Set up hyper-parameters -->
-  <xacro:arg name="prefix" default="right" />
   <xacro:property name="palm_length" value="0.1" />
   <xacro:property name="palm_width" value="0.01" />
@@ -178,5 +180,8 @@
   </xacro:macro>
   <!-- Construct the hand model -->
-  <link name="world" />
+  <xacro:property name="var" value="$(arg parent)" />
+  <xacro:if value="${var == 'world'}">
+    <link name="world" />
+  </xacro:if>
   <!-- Palm -->
   <link name="$(arg prefix)_palm">
@@ -193,5 +198,5 @@
   <joint name="$(arg prefix)_palm_joint" type="fixed">
     <origin xyz="0 0 0" rpy="0 0 0" />
-    <parent link="world" />
+    <parent link="$(arg parent)" />
     <child link="$(arg prefix)_palm" />
   </joint>
