Commit message: Add a human hand model for visualization and later retargeting.

File: arm_hand_retargeting/urdf/human_hand_model.urdf.xacro (robot description, xacro)
@@ -5,6 +5,10 @@
   <xacro:arg name="prefix" default="right" />
   <xacro:property name="palm_length" value="0.1" />
-  <xacro:property name="palm_width" value="0.02" />
-  <xacro:property name="palm_height" value="0.3" />
+  <xacro:property name="palm_width" value="0.01" />
+  <xacro:property name="palm_height" value="0.15" />
+  <!-- Just for visualiation -->
+  <xacro:property name="finger_width" value="0.01" />
+  <xacro:property name="finger_length" value="0.015" />
+  <!-- Macro for three-link *FINGER* model -->
   <xacro:macro name="three_link_finger" params="prefix
                                                 parent
@@ -21,4 +25,7 @@
           <box size="${PP_width} ${PP_length} ${PP_height}" />
         </geometry>
+        <material name="PaleGreen">
+          <color rgba="0.596 0.984 0.596 1.0" />
+        </material>
       </visual>
     </link>
@@ -32,4 +39,7 @@
           <box size="${IP_width} ${IP_length} ${IP_height}" />
         </geometry>
+        <material name="LightSkyBlue">
+          <color rgba="0.529 0.808 0.980 1.0" />
+        </material>
       </visual>
     </link>
@@ -41,4 +51,7 @@
           <box size="${DP_width} ${DP_length} ${DP_height}" />
         </geometry>
+        <material name="LightSalmon">
+          <color rgba="1.0 0.627 0.478 1.0" />
+        </material>
       </visual>
     </link>
@@ -76,6 +89,95 @@
     </joint>
   </xacro:macro>
+  <!-- Macro for three-link *THUMB* model -->
+  <xacro:macro name="three_link_thumb" params="prefix
+                                                parent
+                                                origin_x origin_y origin_z
+                                                DP_length DP_width DP_height
+                                                IP_length IP_width IP_height
+                                                PP_length PP_width PP_height
+                                                ">
+    <!-- virtual links -->
+    <link name="${prefix}_virtual_link_1" />
+    <link name="${prefix}_virtual_link_2" />
+    <!-- Proximal Phalange -->
+    <link name="${prefix}_PP_link">
+      <visual>
+        <origin xyz="0 0 ${PP_height/2}" rpy="0 0 0" />
+        <geometry>
+          <box size="${PP_width} ${PP_length} ${PP_height}" />
+        </geometry>
+        <material name="PaleGreen">
+          <color rgba="0.596 0.984 0.596 1.0" />
+        </material>
+      </visual>
+    </link>
+    <!-- Intermediate Phalange -->
+    <link name="${prefix}_IP_link">
+      <visual>
+        <origin xyz="0 0 ${IP_height/2}" rpy="0 0 0" />
+        <geometry>
+          <box size="${IP_width} ${IP_length} ${IP_height}" />
+        </geometry>
+        <material name="LightSkyBlue">
+          <color rgba="0.529 0.808 0.980 1.0" />
+        </material>
+      </visual>
+    </link>
+    <!-- Distal Phalange -->
+    <link name="${prefix}_DP_link">
+      <visual>
+        <origin xyz="0 0 ${DP_height/2}" rpy="0 0 0" />
+        <geometry>
+          <box size="${DP_width} ${DP_length} ${DP_height}" />
+        </geometry>
+        <material name="LightSalmon">
+          <color rgba="1.0 0.627 0.478 1.0" />
+        </material>
+      </visual>
+    </link>
+    <!-- Metacarpophalangeal Joint 1 -->
+    <joint name="${prefix}_MCP_joint_1" type="revolute">
+      <origin xyz="${origin_x} ${origin_y} ${origin_z}" rpy="0 0 0" />
+      <axis xyz="-1 0 0" />
+      <parent link="${parent}" />
+      <child link="${prefix}_virtual_link_1" />
+      <limit effort="100" velocity="10.0" lower="0.0" upper="${pi/9}" />
+    </joint>
+    <!-- Metacarpophalangeal Joint 2 -->
+    <joint name="${prefix}_MCP_joint_2" type="revolute">
+      <origin xyz="0 0 0" rpy="0 0 0" />
+      <axis xyz="0 0 -1" />
+      <parent link="${prefix}_virtual_link_1" />
+      <child link="${prefix}_PP_link" />
+      <limit effort="100" velocity="10.0" lower="0" upper="${pi/1.8}" />
+    </joint>
+    <!-- Proximal Interphalangeal Joint 1 -->
+    <joint name="${prefix}_PIP_joint_1" type="revolute">
+      <origin xyz="0 0 ${PP_height}" rpy="0 0 0" />
+      <axis xyz="1 0 0" />
+      <parent link="${prefix}_PP_link" />
+      <child link="${prefix}_virtual_link_2" />
+      <limit effort="100" velocity="10.0" lower="0" upper="${pi/4}" />
+    </joint>
+    <!-- Proximal Interphalangeal Joint 2 -->
+    <joint name="${prefix}_PIP_joint_2" type="revolute">
+      <origin xyz="0 0 0" rpy="0 0 0" />
+      <axis xyz="0 1 0" />
+      <parent link="${prefix}_virtual_link_2" />
+      <child link="${prefix}_IP_link" />
+      <limit effort="100" velocity="10.0" lower="0" upper="${pi/2}" />
+    </joint>
+    <!-- Distal Interphalangeal Joint -->
+    <joint name="${prefix}_DIP_joint" type="revolute">
+      <origin xyz="0 0 ${IP_height}" rpy="0 0 0" />
+      <axis xyz="0 1 0" />
+      <parent link="${prefix}_IP_link" />
+      <child link="${prefix}_DP_link" />
+      <limit effort="100" velocity="10.0" lower="0" upper="${pi/2}" />
+    </joint>
+  </xacro:macro>
   <!-- Construct the hand model -->
   <link name="world" />
+  <!-- Palm -->
   <link name="$(arg prefix)_palm">
     <visual>
@@ -84,6 +186,6 @@
         <box size="${palm_width} ${palm_length} ${palm_height}" />
       </geometry>
-      <material name="Cyan">
-        <color rgba="0 1.0 1.0 1.0" />
+      <material name="LightGold">
+        <color rgba="0.933 0.867 0.510 1.0" />
       </material>
     </visual>
@@ -94,8 +196,30 @@
     <child link="$(arg prefix)_palm" />
   </joint>
+  <!-- Four fingers -->
   <xacro:three_link_finger prefix="$(arg prefix)_little_finger" parent="$(arg prefix)_palm"
-                           origin_x="0.0" origin_y="${-palm_length/2}" origin_z="${palm_height}"
-                           DP_length="0.02" DP_width="0.02" DP_height="0.05"
-                           IP_length="0.02" IP_width="0.02" IP_height="0.05"
-                           PP_length="0.02" PP_width="0.02" PP_height="0.05" />
+                           origin_x="0.0" origin_y="${-palm_length/2+finger_length/2}" origin_z="${palm_height}"
+                           DP_length="${finger_length}" DP_width="${finger_width}" DP_height="0.01"
+                           IP_length="${finger_length}" IP_width="${finger_width}" IP_height="0.02"
+                           PP_length="${finger_length}" PP_width="${finger_width}" PP_height="0.03" />
+  <xacro:three_link_finger prefix="$(arg prefix)_ring_finger" parent="$(arg prefix)_palm"
+                           origin_x="0.0" origin_y="${-finger_length/2-0.01}" origin_z="${palm_height}"
+                           DP_length="${finger_length}" DP_width="${finger_width}" DP_height="0.02"
+                           IP_length="${finger_length}" IP_width="${finger_width}" IP_height="0.03"
+                           PP_length="${finger_length}" PP_width="${finger_width}" PP_height="0.04" />
+  <xacro:three_link_finger prefix="$(arg prefix)_middle_finger" parent="$(arg prefix)_palm"
+                           origin_x="0.0" origin_y="${finger_length/2 + 0.01}" origin_z="${palm_height}"
+                           DP_length="${finger_length}" DP_width="${finger_width}" DP_height="0.021"
+                           IP_length="${finger_length}" IP_width="${finger_width}" IP_height="0.032"
+                           PP_length="${finger_length}" PP_width="${finger_width}" PP_height="0.043" />
+  <xacro:three_link_finger prefix="$(arg prefix)_index_finger" parent="$(arg prefix)_palm"
+                           origin_x="0.0" origin_y="${palm_length/2-finger_length/2}" origin_z="${palm_height}"
+                           DP_length="${finger_length}" DP_width="${finger_width}" DP_height="0.02"
+                           IP_length="${finger_length}" IP_width="${finger_width}" IP_height="0.03"
+                           PP_length="${finger_length}" PP_width="${finger_width}" PP_height="0.04" />
+  <!-- Thumb -->
+  <xacro:three_link_thumb prefix="$(arg prefix)_thumb" parent="$(arg prefix)_palm"
+                           origin_x="0.0" origin_y="${palm_length/2}" origin_z="0.0"
+                           DP_length="${finger_length}" DP_width="${finger_width}" DP_height="0.02"
+                           IP_length="${finger_length}" IP_width="${finger_width}" IP_height="0.03"
+                           PP_length="${finger_length}" PP_width="${finger_width}" PP_height="0.05" />
 </robot>

Commit message: Modify the urdf xacro file of human hand model for ease of use.
  - Can easily specify the ref link to which the hand is attached.
  - But the difference in the structures of both hands are not dealt with yet.

File: arm_hand_retargeting/urdf/human_hand_model.urdf.xacro (robot description, xacro)
@@ -2,14 +2,4 @@
 <robot xmlns:xacro="http://wiki.ros.org/xacro"
              name="human_hand_model" >
-  <!-- Configurable arguments -->
-  <xacro:arg name="prefix" default="right" />
-  <xacro:arg name="parent" default="world" />
-  <!-- Set up hyper-parameters -->
-  <xacro:property name="palm_length" value="0.1" />
-  <xacro:property name="palm_width" value="0.01" />
-  <xacro:property name="palm_height" value="0.15" />
-  <!-- Just for visualiation -->
-  <xacro:property name="finger_width" value="0.01" />
-  <xacro:property name="finger_length" value="0.015" />
   <!-- Macro for three-link *FINGER* model -->
   <xacro:macro name="three_link_finger" params="prefix
@@ -179,52 +169,67 @@
     </joint>
   </xacro:macro>
-  <!-- Construct the hand model -->
-  <xacro:property name="var" value="$(arg parent)" />
-  <xacro:if value="${var == 'world'}">
-    <link name="world" />
-  </xacro:if>
-  <!-- Palm -->
-  <link name="$(arg prefix)_palm">
-    <visual>
-      <origin xyz="0 0 ${palm_height/2}" rpy="0 0 0" />
-      <geometry>
-        <box size="${palm_width} ${palm_length} ${palm_height}" />
-      </geometry>
-      <material name="LightGold">
-        <color rgba="0.933 0.867 0.510 1.0" />
-      </material>
-    </visual>
-  </link>
-  <joint name="$(arg prefix)_palm_joint" type="fixed">
-    <origin xyz="0 0 0" rpy="0 0 0" />
-    <parent link="$(arg parent)" />
-    <child link="$(arg prefix)_palm" />
-  </joint>
-  <!-- Four fingers -->
-  <xacro:three_link_finger prefix="$(arg prefix)_little_finger" parent="$(arg prefix)_palm"
-                           origin_x="0.0" origin_y="${-palm_length/2+finger_length/2}" origin_z="${palm_height}"
-                           DP_length="${finger_length}" DP_width="${finger_width}" DP_height="0.01"
-                           IP_length="${finger_length}" IP_width="${finger_width}" IP_height="0.02"
-                           PP_length="${finger_length}" PP_width="${finger_width}" PP_height="0.03" />
-  <xacro:three_link_finger prefix="$(arg prefix)_ring_finger" parent="$(arg prefix)_palm"
-                           origin_x="0.0" origin_y="${-finger_length/2-0.01}" origin_z="${palm_height}"
-                           DP_length="${finger_length}" DP_width="${finger_width}" DP_height="0.02"
-                           IP_length="${finger_length}" IP_width="${finger_width}" IP_height="0.03"
-                           PP_length="${finger_length}" PP_width="${finger_width}" PP_height="0.04" />
-  <xacro:three_link_finger prefix="$(arg prefix)_middle_finger" parent="$(arg prefix)_palm"
-                           origin_x="0.0" origin_y="${finger_length/2 + 0.01}" origin_z="${palm_height}"
-                           DP_length="${finger_length}" DP_width="${finger_width}" DP_height="0.021"
-                           IP_length="${finger_length}" IP_width="${finger_width}" IP_height="0.032"
-                           PP_length="${finger_length}" PP_width="${finger_width}" PP_height="0.043" />
-  <xacro:three_link_finger prefix="$(arg prefix)_index_finger" parent="$(arg prefix)_palm"
-                           origin_x="0.0" origin_y="${palm_length/2-finger_length/2}" origin_z="${palm_height}"
-                           DP_length="${finger_length}" DP_width="${finger_width}" DP_height="0.02"
-                           IP_length="${finger_length}" IP_width="${finger_width}" IP_height="0.03"
-                           PP_length="${finger_length}" PP_width="${finger_width}" PP_height="0.04" />
-  <!-- Thumb -->
-  <xacro:three_link_thumb prefix="$(arg prefix)_thumb" parent="$(arg prefix)_palm"
-                           origin_x="0.0" origin_y="${palm_length/2}" origin_z="0.0"
-                           DP_length="${finger_length}" DP_width="${finger_width}" DP_height="0.02"
-                           IP_length="${finger_length}" IP_width="${finger_width}" IP_height="0.03"
-                           PP_length="${finger_length}" PP_width="${finger_width}" PP_height="0.05" />
+  <!-- Construct the human hand model -->
+  <xacro:macro name="human_hand_model" params="prefix:=right parent:=world">
+    <!-- Configurable arguments -->
+    <!--xacro:arg name="prefix" default="right" /-->
+    <!--xacro:arg name="parent" default="world" /-->
+    <!-- Set up hyper-parameters -->
+    <xacro:property name="palm_length" value="0.1" />
+    <xacro:property name="palm_width" value="0.01" />
+    <xacro:property name="palm_height" value="0.15" />
+    <!-- Just for visualiation -->
+    <xacro:property name="finger_width" value="0.01" />
+    <xacro:property name="finger_length" value="0.015" />
+    <!-- Interval distance between fingers -->
+    <xacro:property name="interval" value="${(palm_length - 4 * finger_length) / 3}" />
+    <!-- Construct the hand model -->
+    <!--xacro:property name="var" value="$(arg parent)" /-->
+    <!--xacro:if value="${parent == 'world'}">
+      <link name="world" />
+    </xacro:if-->
+    <!-- Palm -->
+    <link name="${prefix}_palm">
+      <visual>
+        <origin xyz="0 0 ${palm_height/2}" rpy="0 0 0" />
+        <geometry>
+          <box size="${palm_width} ${palm_length} ${palm_height}" />
+        </geometry>
+        <material name="LightGold">
+          <color rgba="0.933 0.867 0.510 1.0" />
+        </material>
+      </visual>
+    </link>
+    <joint name="${prefix}_palm_joint" type="fixed">
+      <origin xyz="0 0 0" rpy="0 0 0" />
+      <parent link="${parent}" />
+      <child link="${prefix}_palm" />
+    </joint>
+    <!-- Four fingers -->
+    <xacro:three_link_finger prefix="${prefix}_little_finger" parent="${prefix}_palm"
+                             origin_x="0.0" origin_y="${-3*(finger_length+interval)/2}" origin_z="${palm_height}"
+                             DP_length="${finger_length}" DP_width="${finger_width}" DP_height="0.01"
+                             IP_length="${finger_length}" IP_width="${finger_width}" IP_height="0.02"
+                             PP_length="${finger_length}" PP_width="${finger_width}" PP_height="0.03" />
+    <xacro:three_link_finger prefix="${prefix}_ring_finger" parent="${prefix}_palm"
+                             origin_x="0.0" origin_y="${-(finger_length+interval)/2}" origin_z="${palm_height}"
+                             DP_length="${finger_length}" DP_width="${finger_width}" DP_height="0.02"
+                            IP_length="${finger_length}" IP_width="${finger_width}" IP_height="0.03"
+                             PP_length="${finger_length}" PP_width="${finger_width}" PP_height="0.04" />
+    <xacro:three_link_finger prefix="${prefix}_middle_finger" parent="${prefix}_palm"
+                             origin_x="0.0" origin_y="${(finger_length+interval)/2}" origin_z="${palm_height}"
+                             DP_length="${finger_length}" DP_width="${finger_width}" DP_height="0.021"
+                             IP_length="${finger_length}" IP_width="${finger_width}" IP_height="0.032"
+                             PP_length="${finger_length}" PP_width="${finger_width}" PP_height="0.043" />
+    <xacro:three_link_finger prefix="${prefix}_index_finger" parent="${prefix}_palm"
+                             origin_x="0.0" origin_y="${3*(finger_length+interval)/2}" origin_z="${palm_height}"
+                             DP_length="${finger_length}" DP_width="${finger_width}" DP_height="0.02"
+                             IP_length="${finger_length}" IP_width="${finger_width}" IP_height="0.03"
+                             PP_length="${finger_length}" PP_width="${finger_width}" PP_height="0.04" />
+    <!-- Thumb -->
+    <xacro:three_link_thumb prefix="${prefix}_thumb" parent="${prefix}_palm"
+                            origin_x="0.0" origin_y="${palm_length/2}" origin_z="0.0"
+                            DP_length="${finger_length}" DP_width="${finger_width}" DP_height="0.02"
+                            IP_length="${finger_length}" IP_width="${finger_width}" IP_height="0.03"
+                            PP_length="${finger_length}" PP_width="${finger_width}" PP_height="0.05" />
+  </xacro:macro>
 </robot>

Commit message: Test the code for loading visualization markers, and record .bag data of right hand's motion for retargeting experiment.
  - Fail to load the urdf model of human hand into real-time visualization.
  - Re-modify the urdf model for easier use.

File: arm_hand_retargeting/urdf/human_hand_model.urdf.xacro (robot description, xacro)
@@ -184,4 +184,5 @@
     <xacro:property name="interval" value="${(palm_length - 4 * finger_length) / 3}" />
     <!-- Construct the hand model -->
+    <link name="${parent}" />
     <!--xacro:property name="var" value="$(arg parent)" /-->
     <!--xacro:if value="${parent == 'world'}">

File: arm_hand_retargeting/urdf/upload_both_hands.urdf.xacro (robot description, xacro)
@@ -3,6 +3,8 @@
              name="human_hand_model" >
   <xacro:include filename="$(find arm_hand_retargeting)/urdf/human_hand_model.urdf.xacro" />
-  <link name="world" />
-  <xacro:human_hand_model prefix="right" parent="world" />
-  <!--xacro:human_hand_model prefix="left" parent="world" /-->
+  <!-- require a link to attach to -->
+  <!--link name="right_hand" /-->
+  <xacro:human_hand_model prefix="right" parent="right_hand" />
+  <!--link name="left_hand" /-->
+  <xacro:human_hand_model prefix="left" parent="left_hand" />
 </robot>
