Commit message: Implement visualization code for human IK results and for YuMi execting manually mapped human joint trajectories.

File: human_model/urdf/human_model.urdf.xacro (robot description, xacro)
@@ -11,6 +11,6 @@
     <!-- Human upperarm, forearm, hand size parameters -->
     <xacro:property name="arm_scale" value="1"/>
-    <xacro:property name="upperarm_length" value="${0.2*arm_scale}"/>
-    <xacro:property name="forearm_length" value="${0.23*arm_scale}"/>
+    <xacro:property name="upperarm_length" value="0.1850"/> <!--"${0.2*arm_scale}"/-->
+    <xacro:property name="forearm_length" value="0.2264" /> <!--"${0.23*arm_scale}"/-->
     <xacro:property name="hand_length" value="${0.12*arm_scale}"/>
     <xacro:property name="shoulder_height" value="1.3"/>
