Commit message: Modify shadowhand URDF for better visualization. Add batch_process.py for processing dataglove calibration data automatically.

File: dataglove_calib_visual/sr_description/robots/bimanual_shadowhand_motor.urdf.xacro (robot description, xacro)
@@ -8,7 +8,8 @@
     <parent link="world" />
     <child link="rh_forearm" />
-    <origin xyz="0.0 0.0 0.0" rpy="0.0 0.0 0.0" />
+    <!--origin xyz="0.0 0.0 0.0" rpy="0.0 0.0 0.0" /-->
+    <origin xyz="-0.2 0.0 0.0" rpy="0.0 0.0 0.0" /> <!-- Modified by LYW, 2020-11-04 -->
   </joint>
-  <xacro:shadowhand muscletrans="false" muscle="false" bio="false" bt_sp="false"
+  <xacro:shadowhand muscletrans="false" muscle="false" bio="true" bt_sp="false"
   ubi="false" eli="false" reflect="1.0" prefix="rh_" lf="true" />
   <joint name="right_hand_to_left_hand" type="fixed">
@@ -17,5 +18,5 @@
     <origin xyz="0.4 0.0 0.0" rpy="0.0 0.0 0.0" />
   </joint>
-  <xacro:shadowhand muscletrans="false" muscle="false" bio="false" bt_sp="false"
+  <xacro:shadowhand muscletrans="false" muscle="false" bio="true" bt_sp="false"
   ubi="false" eli="false" reflect="-1.0" prefix="lh_" lf="true" />
 </robot>
